Commit message: aggiunta descrizione urdf

File: description/diff_wheeled_robot.xacro (robot description, xacro)
@@ -92,5 +92,5 @@
       <origin xyz="0 0 0" rpy="0 0 0" />
       <geometry>
-        <box size="${hokuyo_size} ${hokuyo_size} ${hokuyo_size}"/>
+        <box size="${kinect_length} ${kinect_height} ${kinect_width}"/>
       </geometry>
       <material name="Blue" />
@@ -98,7 +98,7 @@
   </link>
   <joint name="hokuyo_joint" type="fixed">
-    <origin xyz="${base_radius - hokuyo_size/2} 0 ${base_height+hokuyo_size/4}" rpy="0 0 0" />
+    <origin xyz="${base_radius - kinect_length/2} 0 ${base_height+kinect_height/4}" rpy="0 0 0" />
     <parent link="base_link"/>
-    <child link="hokuyo_link" />
+    <child link="kinect_link" />
   </joint>
 </robot>

File: description/wheel.urdf.xacro (robot description, xacro)
@@ -2,6 +2,6 @@
 <robot name="wheel" xmlns:xacro="http://www.ros.org/wiki/xacro">
   <!-- Wheels -->
-  <property name="wheel_radius" value="0.04" />
-  <property name="wheel_height" value="0.02" />
+  <property name="wheel_radius" value="0.033" />
+  <property name="wheel_height" value="0.021" />
   <property name="base_x_origin_to_wheel_origin" value="0.25" />
   <property name="base_y_origin_to_wheel_origin" value="0.3" />
@@ -10,5 +10,5 @@
     <link name="${lr}_wheel">
       <visual>
-        <origin xyz="0 0 0" rpy="${flipY*M_PI/2} 0  0 " />
+        <origin xyz="0 0 0" rpy="${M_PI/2} 0  0 " />
         <geometry>
           <cylinder length="${wheel_height}" radius="${wheel_radius}" />
@@ -19,5 +19,5 @@
     <joint name="${lr}_wheel_joint" type="continuous">
       <parent link="${parent}"/>
-      <child link="$${lr}_wheel"/>
+      <child link="${lr}_wheel"/>
       <origin xyz="${translateX * base_x_origin_to_wheel_origin} ${translateY * base_y_origin_to_wheel_origin} ${base_z_origin_to_wheel_origin}" rpy="0 0 0" />
       <axis xyz="0 1 0" rpy="0 0 0" />
