Commit message: aggiornamento pdf tf tree

File: description/eod_generated.urdf (robot description, URDF)
Before this commit: robot eod, 6 links, 5 joints
Links:
- added link tower_link; visual box size=0.027 0.072 0.225
- link base_link: geometry visual box size=0.212 0.1 0.033
- link caster_link: geometry visual sphere radius=0.0225
- link kinect_link: geometry visual box size=0.07 0.28 0.07
- link left_wheel: geometry visual cylinder length=0.021 radius=0.033
- link right_wheel: geometry visual cylinder length=0.021 radius=0.033
Joints:
- added joint tower_joint: type fixed, parent base_link, child tower_link, origin xyz=-0.1185 0.0 0.1575 rpy=0 0 0
- joint base_footprint_joint: origin xyz=0 0 0.04 rpy=0 0 0 -> xyz=0 0 0.033 rpy=0 0 0
- joint caster_joint: origin xyz=0.07 0.0 0.007 rpy=-1.57079632679 0 0 -> xyz=-0.115 0.0 0 rpy=0 0 0
- joint kinect_joint: origin xyz=0.075 0 0.05 rpy=0 0 0 -> xyz=0 0 0.1655 rpy=0 0 0; parent base_link -> tower_link

Commit message: Da pc Antonio - 7 Maggio
Ultima configurazione funzionante per il nav stack. Aggiunto nodo per la gestione dei goal

File: description/eod_generated.urdf (robot description, URDF)
Before this commit: robot eod, 9 links, 8 joints
Joints:
- joint camera_joint: origin xyz=0 0 0.1475 rpy=0 0 0 -> xyz=0.027 0 0.1445 rpy=0 0.523598775598 0

File: description/kinect.xacro (robot description, xacro)
@@ -1,13 +1,17 @@
 <?xml version="1.0"?>
 <robot name="sensor_kinect" xmlns:xacro="http://ros.org/wiki/xacro">
-  <xacro:include filename="/opt/ros/indigo/share/turtlebot_description/urdf/turtlebot_gazebo.urdf.xacro"/>
-  <xacro:include filename="/opt/ros/indigo/share/turtlebot_description/urdf/turtlebot_properties.urdf.xacro"/>
+  <xacro:include filename="/opt/ros/kinetic/share/turtlebot_description/urdf/turtlebot_gazebo.urdf.xacro"/>
+  <xacro:include filename="/opt/ros/kinetic/share/turtlebot_description/urdf/turtlebot_properties.urdf.xacro"/>
+  <property name="PI" value="3.1415926535897931" />
   <xacro:property name="kinect_cam_py" value="-0.0125"/>
   <property name="kinect_base_height" value="0.035"/>
   <property name="tower_height" value="0.225" />
+  <property name="tower_length" value="0.027" />
+  <!-- piccola quantita' per far andare la kinect inclinata sulla torretta-->
+  <property name="bias" value="0.003" />
   <!-- Parameterised in part by the values in turtlebot_properties.urdf.xacro -->
   <xacro:macro name="sensor_kinect" params="parent">
     <joint name="camera_joint" type="fixed">
-      <origin xyz="0 0 ${ tower_height/2 + kinect_base_height}" rpy="0 0 0"/>
+      <origin xyz="${tower_length} 0 ${ tower_height/2 + kinect_base_height }" rpy="0 0 0"/>
       <parent link="${parent}"/>
       <child link="camera_link"/>
