Commit message: descrizione con kinect correttamente posizionata

File: description/eod.xacro (robot description, xacro)
@@ -2,4 +2,5 @@
 <robot name="eod" xmlns:xacro="http://www.ros.org/wiki/xacro">
   <xacro:include filename="$(find eod_pkg)/description/wheel.urdf.xacro" />
+  <xacro:include filename="$(find eod_pkg)/description/kinect.xacro" />
 <!-- Defining the colors used in this robot -->
   <material name="Black">
@@ -26,5 +27,5 @@
   <property name="base_length" value="0.212" />
   <property name="back_base_offset" value="0.08" />
-  <property name="height_from_floor" value="0.045" />
+  <property name="height_from_floor" value="0.043" />
   <!-- distanza tra i centri delle due ruote -->
   <property name="l" value="0.135" />
@@ -47,9 +48,9 @@
   <property name="caster_to_back" value="0.017" />
   <!-- Kinect dimensions   -->
-  <property name="kinect_height" value="0.07" />
+  <!--property name="kinect_height" value="0.07" />
   <property name="kinect_width" value="0.28" />
-  <property name="kinect_length" value="0.07" />
+  <property name="kinect_length" value="0.07" /-->
   <!-- presunta altezza del sistema di riferimento della kinect -->
-  <property name="kinect_focus_height" value="0.053" />
+  <!--property name="kinect_focus_height" value="0.053" /-->
   <!-- Wheels -->
   <!--property name="base_x_origin_to_wheel_origin" value="0.25" />
@@ -117,5 +118,5 @@
   <!-- SENSORS -->
   <!-- Kinect -->
-  <link name="kinect_link">
+  <!--link name="kinect_link">
     <visual>
       <origin xyz="0 0 ${-(kinect_height-kinect_focus_height)}" rpy="0 0 0" />
@@ -130,4 +131,5 @@
     <parent link="tower_link"/>
     <child link="kinect_link" />
-  </joint>
+  </joint-->
+  <sensor_kinect parent="tower_link" />
 </robot>

File: description/eod_generated.urdf (robot description, URDF)
Before this commit: robot eod, 7 links, 6 joints
Links:
- removed link kinect_link
- added link camera_link, mass 0.564; collision box size=0.07271 0.27794 0.073; visual mesh filename=package://turtlebot_description/meshes/sensors/kinect.dae
- added link camera_rgb_frame
- added link camera_rgb_optical_frame
- link caster_link: geometry visual sphere radius=0.0215
Joints:
- removed joint kinect_joint
- added joint camera_joint: type fixed, parent tower_link, child camera_link, origin xyz=0 0 0.1475 rpy=0 0 0
- added joint camera_rgb_joint: type fixed, parent camera_link, child camera_rgb_frame, origin xyz=0.031 -0.0125 0.016 rpy=0 0 0
- added joint camera_rgb_optical_joint: type fixed, parent camera_rgb_frame, child camera_rgb_optical_frame, origin xyz=0 0 0 rpy=-1.57079632679 0 -1.57079632679

Commit message: Da pc Antonio - 7 Maggio (2)
AUltima configurazione funzionante per il nav stack. Aggiunto nodo per la gestione dei goal. URDF aggiornato con base_arm

File: description/eod.xacro (robot description, xacro)
@@ -83,4 +83,22 @@
     </visual>
   </link>
+  <!-- BASE-ARM -->
+  <!-- base_arm descrive la posizione del sistema di riferimento base del braccio rispetto a base_link -->
+  <property name="arm_x_offset" value="0.01" />
+  <property name="arm_y_offset" value="0.0" />
+  <property name="arm_z_offset" value="0.04" />
+  <link name="base_arm">
+    <visual>
+        <origin xyz="0 0 0" rpy="0 0 0" />
+        <geometry>
+            <box size="0.001 0.001 0.001" />
+        </geometry>
+    </visual>
+  </link>
+  <joint name="arm_joint" type="fixed">
+    <origin xyz="${arm_x_offset} ${arm_y_offset} ${r_base_offset + arm_z_offset}" rpy="0 0 0" />
+    <parent link="base_link"/>
+    <child link="base_arm" />
+  </joint>
  <!-- TOWER-LINK -->
   <link name="tower_link">

File: description/kinect.xacro (robot description, xacro)
@@ -13,5 +13,5 @@
   <xacro:macro name="sensor_kinect" params="parent">
     <joint name="camera_joint" type="fixed">
-      <origin xyz="${tower_length} 0 ${ tower_height/2 + kinect_base_height }" rpy="0 0 0"/>
+      <origin xyz="0 0 ${ tower_height/2 + kinect_base_height }" rpy="0 0 0"/>
       <parent link="${parent}"/>
       <child link="camera_link"/>

Commit message: Stato: apparentemente funzionante
Aggiunti i file relativi all'identificazione dei motori nuovi.  Aggiunte le foto degli oggetti da identificare. Eliminato il 'bias' da ref_transformer. Aggiunto un parametro importante per il nodo robot_state_publisher. La macchina a stati funziona quasi completamente: bisogna gestire degli offset opportuni e testare completamente il braccio.

File: description/eod.xacro (robot description, xacro)
@@ -38,5 +38,5 @@
   <property name="tower_length" value="0.027" />
   <!-- wheel radius and height -->
-  <property name="wheel_radius" value="0.033" />
+  <property name="wheel_radius" value="0.035" />
   <property name="wheel_height" value="0.021" />
   <property name="wheel_to_front" value="0.08" />
@@ -85,7 +85,7 @@
   <!-- BASE-ARM -->
   <!-- base_arm descrive la posizione del sistema di riferimento base del braccio rispetto a base_link -->
-  <property name="arm_x_offset" value="0.01" />
-  <property name="arm_y_offset" value="0.0" />
-  <property name="arm_z_offset" value="0.04" />
+  <property name="arm_x_offset" value="0.042" />
+  <property name="arm_y_offset" value="0.007" />
+  <property name="arm_z_offset" value="0.002" />
   <link name="base_arm">
     <visual>
@@ -97,5 +97,5 @@
   </link>
   <joint name="arm_joint" type="fixed">
-    <origin xyz="${arm_x_offset} ${arm_y_offset} ${r_base_offset + arm_z_offset}" rpy="0 0 0" />
+    <origin xyz="${arm_x_offset} ${arm_y_offset} ${r_base_offset + base_height + arm_z_offset}" rpy="0 0 ${-M_PI_2}" />
     <parent link="base_link"/>
     <child link="base_arm" />

Commit message: Da Antonio - 19 Maggio
Stato prima del merge finale

File: description/eod.xacro (robot description, xacro)
@@ -38,5 +38,5 @@
   <property name="tower_length" value="0.027" />
   <!-- wheel radius and height -->
-  <property name="wheel_radius" value="0.033" />
+  <property name="wheel_radius" value="0.035" />
   <property name="wheel_height" value="0.021" />
   <property name="wheel_to_front" value="0.08" />
@@ -85,7 +85,7 @@
   <!-- BASE-ARM -->
   <!-- base_arm descrive la posizione del sistema di riferimento base del braccio rispetto a base_link -->
-  <property name="arm_x_offset" value="0.01" />
-  <property name="arm_y_offset" value="0.0" />
-  <property name="arm_z_offset" value="0.04" />
+  <property name="arm_x_offset" value="0.042" />
+  <property name="arm_y_offset" value="0.007" />
+  <property name="arm_z_offset" value="0.002" />
   <link name="base_arm">
     <visual>
@@ -97,5 +97,5 @@
   </link>
   <joint name="arm_joint" type="fixed">
-    <origin xyz="${arm_x_offset} ${arm_y_offset} ${r_base_offset + arm_z_offset}" rpy="0 0 0" />
+    <origin xyz="${arm_x_offset} ${arm_y_offset} ${r_base_offset + base_height +arm_z_offset}" rpy="0 0 ${-M_PI_2}" />
     <parent link="base_link"/>
     <child link="base_arm" />
